Commit message: add oak code and optimizer

File: dex_retargeting/assets/robots/hands/botyard_hand/botyard_hand_left copy 2.urdf (robot description, URDF)
Before this commit: robot dexhand, 33 links, 32 joints
Links:
- added link ee_link
Joints:
- added joint ee_fixed_joint: type fixed, parent palm, child ee_link, origin xyz=0.0 0.0 0.00 rpy=0.0 0.0 0.0
- joint FAJ1: limit lower=-1.5708 upper=1.5708 effort=0.1 velocity=2.0 -> lower=-0.209439510239 upper=0.209439510239 effort=0.1 velocity=2.0
- joint FAJ3: limit lower=-1.5708 upper=1.5708 effort=0.1 velocity=2.0 -> lower=-0.209439510239 upper=0.209439510239 effort=0.1 velocity=2.0
- joint FFJ3: limit lower=-0.261799387799 upper=1.57079632679 effort=0.1 velocity=2.0 -> lower=0.0 upper=1.5708 effort=0.1 velocity=2.0
- joint LFJ3: limit lower=-0.261799387799 upper=1.57079632679 effort=0.1 velocity=2.0 -> lower=0.0 upper=1.5708 effort=0.1 velocity=2.0
- joint LFJ5: limit lower=0 upper=0.785398163397 effort=0.1 velocity=2.0 -> lower=0.0 upper=1.5708 effort=0.1 velocity=2.0
- joint MFJ3: limit lower=-0.261799387799 upper=1.57079632679 effort=0.1 velocity=2.0 -> lower=0.0 upper=1.5708 effort=0.1 velocity=2.0
- joint RFJ3: limit lower=-0.261799387799 upper=1.57079632679 effort=0.1 velocity=2.0 -> lower=0.0 upper=1.5708 effort=0.1 velocity=2.0
- joint THJ1: limit lower=-0.261799387799 upper=1.57079632679 effort=0.1 velocity=2.0 -> lower=0.0 upper=1.5708 effort=0.1 velocity=2.0
- joint THJ2: limit lower=0 upper=0.7854 effort=0.1 velocity=2.0 -> lower=0.0 upper=1.5708 effort=0.1 velocity=2.0
- joint THJ4: limit lower=0.0 upper=1.5708 effort=0.1 velocity=2.0 -> lower=-1.0471975512 upper=1.0471975512 effort=0.1 velocity=2.0
