Commit message: 添加了0角度约束项

File: dex_retargeting/assets/robots/hands/botyard_hand/botyard_hand_left copy 3.urdf (robot description, URDF)
Before this commit: robot dexhand, 33 links, 32 joints
Joints:
- joint FAJ1: limit lower=-0.2618 upper=0.5235 effort=0.1 velocity=2.0 -> lower=-1.5708 upper=1.5708 effort=0.1 velocity=2.0
- joint FAJ3: limit lower=-0.5235 upper=0.5235 effort=0.1 velocity=2.0 -> lower=-1.5708 upper=1.5708 effort=0.1 velocity=2.0
- joint FFJ3: limit lower=0.0 upper=1.5708 effort=0.1 velocity=2.0 -> lower=-0.261799387799 upper=1.57079632679 effort=0.1 velocity=2.0
- joint LFJ3: limit lower=0.0 upper=1.5708 effort=0.1 velocity=2.0 -> lower=0 upper=1.57079632679 effort=0.1 velocity=2.0
- joint LFJ4: limit lower=-0.2616 upper=0.2616 effort=0.1 velocity=2.0 -> lower=-0.1309 upper=0.1309 effort=0.1 velocity=2.0
- joint LFJ5: limit lower=0.0 upper=1.5708 effort=0.1 velocity=2.0 -> lower=0 upper=0.785398163397 effort=0.1 velocity=2.0
- joint MFJ3: limit lower=0.0 upper=1.5708 effort=0.1 velocity=2.0 -> lower=-0.261799387799 upper=1.57079632679 effort=0.1 velocity=2.0
- joint MFJ4: limit lower=-0.2616 upper=0.2616 effort=0.1 velocity=2.0 -> lower=-0.1309 upper=0.1309 effort=0.1 velocity=2.0
- joint RFJ3: limit lower=0.0 upper=1.5708 effort=0.1 velocity=2.0 -> lower=-0.261799387799 upper=1.57079632679 effort=0.1 velocity=2.0
- joint RFJ4: limit lower=-0.2616 upper=0.2616 effort=0.1 velocity=2.0 -> lower=-0.1309 upper=0.1309 effort=0.1 velocity=2.0
- joint THJ1: limit lower=0.0 upper=1.5708 effort=0.1 velocity=2.0 -> lower=-0.261799387799 upper=1.57079632679 effort=0.1 velocity=2.0
- joint THJ3: limit lower=0.0 upper=0.7854 effort=0.1 velocity=2.0 -> lower=0.0 upper=1.5708 effort=0.1 velocity=2.0
- joint THJ4: limit lower=-0.08 upper=1.5708 effort=0.1 velocity=2.0 -> lower=0.0 upper=1.5708 effort=0.1 velocity=2.0
